Commit message: i fell pain

File: urdf/auto_car.urdf (robot description, URDF)
Before this commit: robot auto_car, 4 links, 2 joints
Links:
- removed link ang_link1
- removed link ang_link7
- removed link camera
- removed link odom
- added link base_link; visual mesh filename=package://auto_car/urdf/car.stl scale=0.01 0.01 0.01
Joints:
- removed joint ang_base
- removed joint camera_joint

Commit message: nice day man

File: urdf/auto_car.urdf (robot description, URDF)
Before this commit: robot auto_car, 1 links, 0 joints
Links:
- link base_link: geometry visual mesh filename=package://auto_car/urdf/car1.stl scale=0.001 0.001 0.001
